File: Electronics/RevB/KiCAD/LiControl/LiControl.kicad_pcb (KiCad board)
At the start: 2 copper layers, 41 x 80 mm, 83 parts, among them J1 Conn_01x08, J2 Conn_01x04, J4 Conn_01x08, J5 RJ45, J6 Conn_02x03_Odd_Even, Q10 Q_NMOS_GSD, Q11 Q_PMOS_GSD, Q12 Q_NMOS_GSD, Q2 Q_NMOS_GSD, Q6 Q_NMOS_GSD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

Commit message: RevB PCB
Parts:
- added REF**: OSHW-Logo2_7.3x6mm_SilkScreen, Symbol:OSHW-Logo2_7.3x6mm_SilkScreen, B.Cu at (116.8, 121.0)
- moved R5 35.9 mm to (112.8, 121.8), turned to 270 degrees
- moved R44 29.8 mm to (110.0, 121.8), turned to 90 degrees
- moved R41 23.6 mm to (94.5, 119.5), turned to 180 degrees
- moved R1 16.8 mm to (114.2, 111.5), turned to 180 degrees
- moved D4 16.1 mm to (107.0, 130.8), turned to 270 degrees
- moved J1 15.2 mm to (89.5, 144.2)
- moved R15 12.9 mm to (94.5, 113.0), turned to 180 degrees
- moved C11 12.5 mm to (88.2, 86.5), turned to 180 degrees
- moved R17 12.1 mm to (110.5, 118.0), turned to 315 degrees
- moved D6 11.5 mm to (102.2, 121.2), turned to 90 degrees
- moved C5 11.5 mm to (106.0, 112.2), turned to 270 degrees
- moved HS1 11.5 mm to (106.2, 131.8), turned to 0 degrees
- moved R9 10.3 mm to (106.5, 115.8), turned to 0 degrees
- moved R11 9.50 mm to (94.5, 116.2), turned to 0 degrees
- moved R4 8.75 mm to (102.5, 112.5), turned to 0 degrees
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Routing:
- net GND: track 65.3 -> 265.6 mm, vias 2 -> 22
- net +5V: track 27.9 -> 151.3 mm, vias 0 -> 7
- net /CLUTCH_uC: track 0.00 -> 65.3 mm, vias 0 -> 1
- net /MAMODE2_ECM_uC: track 0.00 -> 53.9 mm, vias 0 -> 1
- net /MAP_uC: track 0.00 -> 52.9 mm, vias 0 -> 2
- net /BRAKE_RAW: track 18.4 -> 62.7 mm, vias 0 -> 7
- net /12V_ALWAYS: track 0.00 -> 42.6 mm
- net /BRAKE_uC: track 0.00 -> 39.5 mm, vias 0 -> 1
- net /VSS: track 19.6 -> 55.7 mm, vias 1 -> 0
- net /BRAKE_DRIVE: track 0.00 -> 35.4 mm
- net /MODE_SEL2: track 0.00 -> 34.2 mm
- net /CMDPWR_ECM: track 0.00 -> 29.9 mm, vias 0 -> 1
- net /BUTTON: track 0.00 -> 26.1 mm
- net /VSS_PCINT2: track 0.00 -> 26.0 mm
- net /NEP_D: track 19.1 -> 42.1 mm, vias 0 -> 2
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- added copper zone on B.Cu, net +5V
- added copper zone on F.Cu, net +5V
- added copper zone on F.Cu, net /12V_ALWAYS
- added copper zone on F.Cu, net /12V_KEYON
- added copper zone on B.Cu, net /BRAKE_DRIVE
- added copper zone on B.Cu, net /BRAKE_RAW
- added copper zone on F.Cu, net /BRAKE_RAW
- added copper zone on B.Cu, net GND
- added copper zone on F.Cu, net GND
Other:
- board size 41 x 80 mm -> 41 x 79.2 mm
- board text added: "36-8827-ND MOUNTING HOLE (BACK SIDE)"
- board text added: "<PINOUT (UPPER)"
- board text added: "FRONT"
- board text added: "HONDA INSIGHT MANUAL IMA CONTROLLER"
- board text added: "John Sullivan (aka 'mudder'): github.com/doppelhub/MuddersMIMA"
- board text added: "MAMOD2:BLK/YEL[L22] GNDENG:BRN/YEL[L20] 12VHOT:WHT/BLU[U9] VSS:BLU/WHT[U8] 12VKEY:BLK/YEL[U7] CMDPWR:BLU/BLK[L4] NEP:BLU/BLU[U2] MAMOD1:RED/YEL[L1]"
- board text added: "REAR"
- board text added: "WARNING: HEAT SINK MUST NOT CONTACT CHASSIS! CONNECTS TO +12V WHILE BRAKING"
- board text removed: "36-8827-ND MOUNTING HOLE"
- board text removed: "<<C506 "[U_]""
- board text removed: "BLK/YEL[L22] BRN/YEL[L20] WHT/BLU[U9] BLU/WHT[U8] BLK/YEL[U7] BLU/BLK[L4] BLU/BLU[U2] RED/YEL[L1]"
- board text removed: "MAMOD2 GROUND 12V_HOT VSS 12V_KEY CMDPWR NEP MAMOD1"
- board text removed: "github.com/ doppelhub/ MuddersMIMA"
