File: Electronics/RevB/KiCAD/LiControl/LiControl.sch (KiCad schematic (older format))
At the start: 83 parts, among them J1 Conn_01x08, J2 Conn_01x04, J4 Conn_01x08, J5 RJ45, J6 Conn_02x03_Odd_Even, Q10 Q_NMOS_GSD, Q11 Q_PMOS_GSD, Q12 Q_NMOS_GSD, Q2 Q_NMOS_GSD, Q6 Q_NMOS_GSD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

Commit message: RevB PCB
Other:
- note added: "THERE ARE QTY3 BLK/YEL\nWIRES IN THE HARNESS:\n-QTY2 are +12V_KEYON\n-QTY1 is MAMODE2 (5V)"
- note removed: "THERE ARE QTY3 BLK/YEL\nWIRES IN THE HARNESS:\n-QTY2 are +12V_KEYON\n-QTY1 is MAMODE2"
Changed lines of the file:
@@
 MAMODE2_ECM_VLIM
 Text Notes 8275 3400 0    50   ~ 0
-THERE ARE QTY3 BLK/YEL\nWIRES IN THE HARNESS:\n-QTY2 are +12V_KEYON\n-QTY1 is MAMODE2
+THERE ARE QTY3 BLK/YEL\nWIRES IN THE HARNESS:\n-QTY2 are +12V_KEYON\n-QTY1 is MAMODE2 (5V)
 Wire Wire Line
 	8100 2950 8100 2875
